File: bFlightPCB.sch (KiCad schematic (older format))
At the start: 20 parts, among them SW1 ESC_Pad_D, SW2 ESC_Pad_D, SW3 ESC_Pad_D, SW4 ESC_Pad_D, SW5 ESC_Pad_D, SW6 ESC_Pad_D, U1 WeMos_mini, U2 OLED_I2C_128X64_096IN

Commit message: Updated component on PCB to smaller layout
Parts:
- D1, D2, D3, D4, D5, D6: footprint Diode_THT:D_5KPW_P7.62mm_Vertical_AnodeUp -> Diode_THT:D_DO-35_SOD27_P2.54mm_Vertical_AnodeUp
Changed lines of the file:
@@
 F 0 "D6" V 7254 2229 50  0000 L CNN
 F 1 "D_ALT" V 7345 2229 50  0000 L CNN
-F 2 "Diode_THT:D_5KPW_P7.62mm_Vertical_AnodeUp" H 7300 2150 50  0001 C CNN
+F 2 "Diode_THT:D_DO-35_SOD27_P2.54mm_Vertical_AnodeUp" H 7300 2150 50  0001 C CNN
 F 3 "~" H 7300 2150 50  0001 C CNN
 	1    7300 2150
@@
 F 0 "D5" V 7054 2229 50  0000 L CNN
 F 1 "D_ALT" V 7145 2229 50  0000 L CNN
-F 2 "Diode_THT:D_5KPW_P7.62mm_Vertical_AnodeUp" H 7100 2150 50  0001 C CNN
+F 2 "Diode_THT:D_DO-35_SOD27_P2.54mm_Vertical_AnodeUp" H 7100 2150 50  0001 C CNN
 F 3 "~" H 7100 2150 50  0001 C CNN
 	1    7100 2150
@@
 F 0 "D4" V 4954 2229 50  0000 L CNN
 F 1 "D_ALT" V 5045 2229 50  0000 L CNN
-F 2 "Diode_THT:D_5KPW_P7.62mm_Vertical_AnodeUp" H 5000 2150 50  0001 C CNN
+F 2 "Diode_THT:D_DO-35_SOD27_P2.54mm_Vertical_AnodeUp" H 5000 2150 50  0001 C CNN
 F 3 "~" H 5000 2150 50  0001 C CNN
 	1    5000 2150
@@
 F 0 "D3" V 4804 2229 50  0000 L CNN
 F 1 "D_ALT" V 4895 2229 50  0000 L CNN
-F 2 "Diode_THT:D_5KPW_P7.62mm_Vertical_AnodeUp" H 4850 2150 50  0001 C CNN
+F 2 "Diode_THT:D_DO-35_SOD27_P2.54mm_Vertical_AnodeUp" H 4850 2150 50  0001 C CNN
 F 3 "~" H 4850 2150 50  0001 C CNN
 	1    4850 2150
@@
 F 0 "D2" V 4654 2229 50  0000 L CNN
 F 1 "D_ALT" V 4745 2229 50  0000 L CNN
-F 2 "Diode_THT:D_5KPW_P7.62mm_Vertical_AnodeUp" H 4700 2150 50  0001 C CNN
+F 2 "Diode_THT:D_DO-35_SOD27_P2.54mm_Vertical_AnodeUp" H 4700 2150 50  0001 C CNN
 F 3 "~" H 4700 2150 50  0001 C CNN
 	1    4700 2150
@@
 F 0 "D1" V 4504 2229 50  0000 L CNN
 F 1 "D_ALT" V 4595 2229 50  0000 L CNN
-F 2 "Diode_THT:D_5KPW_P7.62mm_Vertical_AnodeUp" H 4550 2150 50  0001 C CNN
+F 2 "Diode_THT:D_DO-35_SOD27_P2.54mm_Vertical_AnodeUp" H 4550 2150 50  0001 C CNN
 F 3 "~" H 4550 2150 50  0001 C CNN
 	1    4550 2150
